Commit message: Updated readme

File: robominer_description/urdf/mesh/mecanum_wheel.urdf.xacro (robot description, xacro)
@@ -3,5 +3,5 @@
   <xacro:macro name="mecanum_wheel" params="side radius width pos_x pos_y pos_z mass">
     <link name="${side}_wheel_link">
-      <visual>
+      <!-- <visual>
         <origin xyz="0 0 0" rpy="${pi/2} 0 0"/>
         <geometry>
@@ -11,5 +11,5 @@
             <color rgba="0.1764 0.4588 0.8509 1.0"/>
         </material>
-      </visual>
+      </visual> -->
       <collision>
         <origin xyz="0 0 0" rpy="${pi/2} 0 0"/>
@@ -31,5 +31,5 @@
     </gazebo>
     <gazebo reference="${side}_wheel_link">
-      <visual>
+      <!-- <visual>
         <material>
           <ambient>0.1764 0.4588 0.8509 1.0</ambient>
@@ -38,5 +38,5 @@
           <emissive>0.0 0.0 0.0 0.0</emissive>
         </material>
-      </visual>
+      </visual> -->
     </gazebo>
     <joint name="${side}_wheel_joint" type="continuous">
