Commit message: Fixed Screw mesh visualization. Fixed ccw and cw screws in visual tags Simplified geometries to get a higher RT factor TODO: Fix whiskers behaviour

File: RM3_gazebo/urdf/RM3_robot.xacro.urdf (robot description, URDF)
Before this commit: robot RM3_robot, 2 links, 1 joints
Links:
- link chassis: mass 8.0 -> 25; geometry collision box size=${body_collision_box_x} ${body_collision_box_y} ${body_coll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; visual mesh filename=file://$(find rm3_gazebo)/urdf/meshes/body_platform.dae

File: RM3_gazebo/urdf/screw_snippets.xacro (robot description, xacro)
@@ -27,19 +27,20 @@
                  <origin xyz="0.17 0.0 0.0" rpy="0 0.0 0"/>
             </xacro:if>
-          <mass value="1" />
-          <inertia ixx="0.0012" ixy="0.0" ixz="0.0"
-                 iyy="0.00079" iyz="0.0"
-                 izz="0.0079" />
+          <mass value="3" />
+          <inertia ixx="0.0035" ixy="0.0" ixz="0.0"
+                 iyy="0.02376" iyz="0.0"
+                 izz="0.02376" />
        </inertial>
         <visual>
-          <origin xyz="0 0 0" rpy="0 0 0" />
           <xacro:if value="${name == 'FR' or name == 'BL'}">
+              <origin xyz="0 0 0" rpy="0 0 3.14" />
               <geometry>
-                <mesh filename="${cw_mesh_file}" scale="1 1 1"/>
+                <mesh filename="${ccw_mesh_file}" scale="1 1 1"/>
               </geometry>
           </xacro:if>
           <xacro:if value="${name == 'FL' or name == 'BR'}">
+              <origin xyz="0 0 0" rpy="0 0 3.14" />
               <geometry>
-                <mesh filename="${ccw_mesh_file}" scale="1 1 1"/>
+                <mesh filename="${cw_mesh_file}" scale="1 1 1"/>
               </geometry>
           </xacro:if>
@@ -79,10 +80,10 @@
                  <origin xyz="0.17 0.0 0.0" rpy="0 0.0 0"/>
             </xacro:if>
-          <mass value="3" />
-          <inertia ixx="0.0012" ixy="0.0" ixz="0.0"
-                 iyy="0.00079" iyz="0.0"
-                 izz="0.0079" />
+          <mass value="0.0001" />
+          <inertia ixx="1.0e-8" ixy="0.0" ixz="0.0"
+                 iyy="1.0e-8" iyz="0.0"
+                 izz="1.0e-8" />
           </inertial>
-        <collision>
+        <!-- <collision>
            <xacro:if value="${name == 'FR_collision' or name == 'BL_collision'}">
                <geometry>
@@ -95,10 +96,32 @@
                </geometry>
            </xacro:if>
+        </collision> -->
+        <collision>
+            <xacro:if value="${name == 'FR_collision' or name == 'BL_collision'}">
+                <origin xyz="0.15 0.0 0.0" rpy="0 1.57 0"/>
+            </xacro:if>
+            <xacro:if value="${name == 'FL_collision' or name == 'BR_collision'}">
+                <origin xyz="-0.15 0.0 0.0" rpy="0 1.57 0"/>
+            </xacro:if>
+           <geometry>
+             <cylinder radius="0.055" length="${screw_collision_height}"/>
+           </geometry>
+        </collision>
+        <collision>
+            <xacro:if value="${name == 'FR_collision' or name == 'BL_collision'}">
+                <origin xyz="0.25 0.0 0.0" rpy="0 0 0"/>
+            </xacro:if>
+            <xacro:if value="${name == 'FL_collision' or name == 'BR_collision'}">
+                <origin xyz="-0.25 0.0 0.0" rpy="0 0 0"/>
+            </xacro:if>
+           <geometry>
+             <sphere radius="0.055"/>
+           </geometry>
         </collision>
       </link>
       <gazebo reference="${name}_screw_link">
-        <mu1 value="1"/>
-        <mu2 value="1"/>
-        <kp value="100000.0" />
+        <mu1 value="100"/>
+        <mu2 value="2"/>
+        <kp value="10.0" />
         <kd value="1.0" />
         <material>Gazebo/Grey</material>

File: RM3_gazebo/urdf/whisker_snippets.xacro (robot description, xacro)
@@ -9,5 +9,5 @@
   <xacro:property name="whisker_length" value="0.150"/>
   <xacro:property name="whisker_radius" value="0.002"/>
-  <xacro:property name="whisker_body_mass" value="0.015"/>
+  <xacro:property name="whisker_body_mass" value="0.008"/>
   <xacro:property name="base_link_mass" value="0.1"/>
   <xacro:property name="whisker_array_mass" value="2.75"/>
@@ -18,4 +18,9 @@
   <xacro:property name="whisker_y" value="0.001"/>
   <xacro:property name="whisker_z" value="0.02"/>
+  <xacro:property name="whisker_damping" value="0.1"/>
+  <xacro:property name="whisker_friction" value="0.001"/>
+  <xacro:property name="whisker_collision_box_x" value="0.6"/>
+  <xacro:property name="whisker_collision_box_y" value="0.08"/>
+  <xacro:property name="whisker_collision_box_z" value="0.07"/>
  <!-- WHISKER DEFITION -->
   <xacro:macro name="whisker" params="name id parent *origin">
@@ -32,11 +37,11 @@
           velocity="${whisker_revolute_vel_limit}" />
         <dynamics
-          damping="0.1"
-          friction="0.1" />
+          damping="${whisker_damping}"
+          friction="${whisker_friction}" />
         </joint>
         <link name="${name}_magnet_x_link_${id}">
         <inertial>
         <mass value="0.0005" />
-        <inertia ixx="1.0e-4" ixy="0" ixz="0" iyy="1.0e-4" iyz="0" izz="1.0e-4" />
+        <inertia ixx="1.0e-8" ixy="0" ixz="0" iyy="1.0e-8" iyz="0" izz="1.0e-8" />
         </inertial>
         </link>
@@ -52,12 +57,12 @@
           velocity="${whisker_revolute_vel_limit}" />
         <dynamics
-          damping="0.1"
-          friction="0.1" />
+            damping="${whisker_damping}"
+            friction="${whisker_friction}" />
         </joint>
         <link name="${name}_magnet_y_link_${id}">
-        <inertial>
-        <mass value="0.0005" />
-        <inertia ixx="1.0e-4" ixy="0" ixz="0" iyy="1.0e-4" iyz="0" izz="1.0e-4" />
-        </inertial>
+            <inertial>
+            <mass value="0.0005" />
+            <inertia ixx="1.0e-8" ixy="0" ixz="0" iyy="1.0e-8" iyz="0" izz="1.0e-8" />
+            </inertial>
         </link>
       <!-- Whisker fixed on magnet y-->
@@ -70,22 +75,42 @@
       <link name="${name}_whisker_link_${id}">
           <inertial>
+            <origin xyz="0 0 ${whisker_length/2}"
+                      rpy="0 0 0" />
             <mass
               value="${whisker_body_mass}" />
-            <inertia
+            <!-- <inertia
               ixx="${1/12 * whisker_body_mass * (3* whisker_radius ** 2 + whisker_length **2 )}" ixy="0" ixz="0"
               iyy="${1/12 * whisker_body_mass * (3* whisker_radius ** 2 + whisker_length **2 )}" iyz="0"
-              izz="${1/2 * whisker_body_mass * whisker_radius ** 2}" />
+              izz="${1/2 * whisker_body_mass * whisker_radius ** 2}" /> -->
+              <inertia
+                ixx="${(1/12)*whisker_body_mass*(3*whisker_radius*whisker_radius + whisker_length*whisker_length)}" ixy="0" ixz="0"
+                iyy="${(1/12)*whisker_body_mass*(3*whisker_radius*whisker_radius + whisker_length*whisker_length)}" iyz="0"
+                izz="${(1/2)*whisker_body_mass*whisker_radius*whisker_radius}" />
           </inertial>
           <visual>
+              <origin xyz="0 0 ${whisker_length/2}"
+                      rpy="0 0 0" />
               <geometry>
-                <mesh filename="${whisker_mesh_file}" scale="1 1 1"/>
+                <cylinder radius="${whisker_radius}" length="${whisker_length-0.01}"/>
               </geometry>
           </visual>
           <collision>
-               <geometry>
-                 <mesh filename="${whisker_mesh_file}" scale="1 1 1"/>
-               </geometry>
+              <origin xyz="0 0 ${whisker_length/2}"
+                      rpy="0 0 0" />
+              <geometry>
+                <cylinder radius="${whisker_radius}" length="${whisker_length-0.01}"/>
+              </geometry>
           </collision>
       </link>
+      <!-- <gazebo reference="${name}_magnet_x_${id}">
+      <implicitSpringDamper>true</implicitSpringDamper>
+      <springStiffness>10000</springStiffness>
+      <springReference>0.0</springReference>
+      </gazebo>
+      <gazebo reference="${name}_magnet_y_${id}">
+      <implicitSpringDamper>true</implicitSpringDamper>
+      <springStiffness>10000</springStiffness>
+      <springReference>0.0</springReference>
+      </gazebo> -->
   </xacro:macro>
  <!-- WHISKER ARRAY DEFITION -->
@@ -98,10 +123,14 @@
       <link name="${name}_whisker_array_link">
         <inertial>
-          <xacro:insert_block name="origin"/>
+          <!-- <xacro:insert_block name="origin"/> -->
           <mass value="${whisker_array_mass}" />
-          <inertia ixx="0.0012" ixy="0.0" ixz="0.0"
-                 iyy="0.00079" iyz="0.0"
-                 izz="0.0079" />
-          </inertial>
+          <inertia
+            ixx="${(1/12)*whisker_array_mass*(whisker_collision_box_z*whisker_collision_box_z + whisker_collision_box_y*whisker_collision_box_y)}"
+            ixy="0.0"
+            ixz="0.0"
+            iyy="${(1/12)*whisker_array_mass*(whisker_collision_box_z*whisker_collision_box_z + whisker_collision_box_x*whisker_collision_box_x)}"
+            iyz="0.0"
+            izz="${(1/12)*whisker_array_mass*(whisker_collision_box_x*whisker_collision_box_x + whisker_collision_box_y*whisker_collision_box_y)}"/>
+        </inertial>
           <visual>
               <geometry>
@@ -109,9 +138,9 @@
               </geometry>
           </visual>
-        <collision>
-               <geometry>
-                 <mesh filename="${whisker_array_mesh_file}" scale="1 1 1"/>
-               </geometry>
-        </collision>
+          <collision>
+            <geometry>
+              <box size="${whisker_collision_box_x} ${whisker_collision_box_y} ${whisker_collision_box_z}" />
+            </geometry>
+          </collision>
       </link>
       <gazebo reference="${name}_whisker_array_link">
