Commit message: Fixed whiskers behaviour Fixed screw/ground collision behaviour TODO: Tune friction parameters for several types of ground

File: RM3_gazebo/urdf/RM3_robot.xacro.urdf (robot description, URDF)
Before this commit: robot RM3_robot, 2 links, 1 joints
Links:
- link chassis: mass 25 -> ${body_mass}

File: RM3_gazebo/urdf/screw_snippets.xacro (robot description, xacro)
@@ -1,10 +1,11 @@
 <?xml version="1.0"?>
 <robot xmlns:xacro="http://www.ros.org/wiki/xacro">
+  <!-- Mesh files -->
   <xacro:property name="ccw_mesh_file" value="file://$(find rm3_gazebo)/urdf/meshes/screw_ccw.dae"/>
   <xacro:property name="cw_mesh_file" value="file://$(find rm3_gazebo)/urdf/meshes/screw_cw.dae"/>
-  <xacro:property name="screw_collision_radius" value="0.02"/>
-  <xacro:property name="screw_collision_height" value="0.2"/>
-  <xacro:property name="passive_wheel_diam" value="0.14" />
-  <xacro:property name="passive_wheel_mass" value="0.2" />
+  <!-- Collisions and inertial parameters -->
+  <xacro:property name="screw_collision_radius" value="0.055"/>
+  <xacro:property name="screw_collision_height" value="0.48"/>
+  <xacro:property name="screw_mass" value="3.0"/>
   <!-- Screw velocity limits  -->
   <xacro:property name="screw_min_velocity" value="-50"/>
@@ -12,4 +13,6 @@
 <!-- Macro for screw defintion -->
   <xacro:macro name="screw" params="name *origin">
+      <!--  THIS LINK IS USED TO VISUALIZE SCREW ROTATIONS -->
+      <!-- *********************************************** -->
       <joint name="${name}_screw" type="continuous">
           <xacro:insert_block name="origin"/>
@@ -22,13 +25,15 @@
         <inertial>
             <xacro:if value="${name == 'BR' or name == 'FL'}">
-                 <origin xyz="-0.17 0.0 0.0" rpy="0 0.0 0"/>
+                 <origin xyz="-0.17 0.0 0.0" rpy="0 1.57 0"/>
             </xacro:if>
             <xacro:if value="${name == 'FR' or name == 'BL'}">
-                 <origin xyz="0.17 0.0 0.0" rpy="0 0.0 0"/>
+                 <origin xyz="0.17 0.0 0.0" rpy="0 1.57 0"/>
             </xacro:if>
-          <mass value="3" />
-          <inertia ixx="0.0035" ixy="0.0" ixz="0.0"
-                 iyy="0.02376" iyz="0.0"
-                 izz="0.02376" />
+          <mass value="${screw_mass / 100}" />
+          <inertia ixx="${(1.0 / 12.0) * screw_mass / 100 * (3 * screw_collision_radius ** 2 + screw_collision_height **2)}"
+                   iyy="${(1.0 / 12.0) * screw_mass / 100 * (3 * screw_collision_radius ** 2 + screw_collision_height **2)}"
+                   izz="${(1.0 / 12.0) * screw_mass / 100 * screw_collision_radius ** 2}"
+                   iyz="0.0" ixy="0.0" ixz="0.0"
+                    />
        </inertial>
         <visual>
@@ -46,83 +51,56 @@
           </xacro:if>
         </visual>
-        <collision>
-            <xacro:if value="${name == 'FR' or name == 'FL'}">
-                <origin xyz="0.15 0.0 0.0" rpy="0 1.57 0"/>
-            </xacro:if>
-            <xacro:if value="${name == 'BL' or name == 'BR'}">
-                <origin xyz="-0.15 0.0 0.0" rpy="0 1.57 0"/>
-            </xacro:if>
-           <geometry>
-             <cylinder radius="${screw_collision_radius}" length="${screw_collision_height}"/>
-           </geometry>
-        </collision>
       </link>
-      <gazebo reference="${name}_screw_link">
-        <mu1 value="0.0"/>
-        <mu2 value="0.0"/>
-        <kp value="100000.0" />
-        <kd value="1.0" />
-      </gazebo>
-  </xacro:macro>
-   <!-- Macro for screw collision based on passive wheels -->
-  <xacro:macro name="screw_collision" params="name *origin">
-      <joint name="${name}_screw" type="fixed">
+      <!-- *********************************************** -->
+      <!--  THIS LINK IS USED TO ENSURE SIMPLER AND TUNABLE COLLISIONS WITH THE ENVIRONMENT -->
+      <!-- *********************************************** -->
+      <joint name="${name}_screw_collision" type="fixed">
           <xacro:insert_block name="origin"/>
           <parent link="chassis"/>
-          <child link="${name}_screw_link"/>
+          <child link="${name}_screw_collision_link"/>
       </joint>
-      <link name="${name}_screw_link">
+      <link name="${name}_screw_collision_link">
         <inertial>
-            <xacro:if value="${name == 'BR_collision' or name == 'FL_collision'}">
+            <xacro:if value="${name == 'BR' or name == 'FL'}">
                  <origin xyz="-0.17 0.0 0.0" rpy="0 0.0 0"/>
             </xacro:if>
-            <xacro:if value="${name == 'FR_collision' or name == 'BL_collision'}">
+            <xacro:if value="${name == 'FR' or name == 'BL'}">
                  <origin xyz="0.17 0.0 0.0" rpy="0 0.0 0"/>
             </xacro:if>
-          <mass value="0.0001" />
-          <inertia ixx="1.0e-8" ixy="0.0" ixz="0.0"
-                 iyy="1.0e-8" iyz="0.0"
-                 izz="1.0e-8" />
-          </inertial>
-        <!-- <collision>
-           <xacro:if value="${name == 'FR_collision' or name == 'BL_collision'}">
-               <geometry>
-                 <mesh filename="${cw_mesh_file}" scale="1 0.9 0.9"/>
-               </geometry>
-           </xacro:if>
-           <xacro:if value="${name == 'FL_collision' or name == 'BR_collision'}">
-               <geometry>
-                 <mesh filename="${ccw_mesh_file}" scale="1 0.9 0.9"/>
-               </geometry>
-           </xacro:if>
-        </collision> -->
-        <collision>
-            <xacro:if value="${name == 'FR_collision' or name == 'BL_collision'}">
-                <origin xyz="0.15 0.0 0.0" rpy="0 1.57 0"/>
-            </xacro:if>
-            <xacro:if value="${name == 'FL_collision' or name == 'BR_collision'}">
-                <origin xyz="-0.15 0.0 0.0" rpy="0 1.57 0"/>
-            </xacro:if>
-           <geometry>
-             <cylinder radius="0.055" length="${screw_collision_height}"/>
-           </geometry>
-        </collision>
-        <collision>
-            <xacro:if value="${name == 'FR_collision' or name == 'BL_collision'}">
-                <origin xyz="0.25 0.0 0.0" rpy="0 0 0"/>
-            </xacro:if>
-            <xacro:if value="${name == 'FL_collision' or name == 'BR_collision'}">
-                <origin xyz="-0.25 0.0 0.0" rpy="0 0 0"/>
-            </xacro:if>
-           <geometry>
-             <sphere radius="0.055"/>
-           </geometry>
-        </collision>
+            <mass value="${screw_mass}" />
+            <inertia ixx="${(1.0 / 12.0) * screw_mass * (3 * screw_collision_radius ** 2 + screw_collision_height **2)}"
+                     iyy="${(1.0 / 12.0) * screw_mass * (3 * screw_collision_radius ** 2 + screw_collision_height **2)}"
+                     izz="${(1.0 / 12.0) * screw_mass * screw_collision_radius ** 2}"
+                     iyz="0.0" ixy="0.0" ixz="0.0"
+                      />
+         </inertial>
+         <collision>
+             <xacro:if value="${name == 'FR' or name == 'BL'}">
+                 <origin xyz="0.0 0.0 0.0" rpy="0 1.57 0"/>
+             </xacro:if>
+             <xacro:if value="${name == 'FL' or name == 'BR'}">
+                 <origin xyz="-0.0 0.0 0.0" rpy="0 1.57 0"/>
+             </xacro:if>
+            <geometry>
+              <cylinder radius="${screw_collision_radius}" length="${screw_collision_height}"/>
+            </geometry>
+         </collision>
+         <collision>
+             <xacro:if value="${name == 'FR' or name == 'BL'}">
+                 <origin xyz="0.25 0.0 0.0" rpy="0 0 0"/>
+             </xacro:if>
+             <xacro:if value="${name == 'FL' or name == 'BR'}">
+                 <origin xyz="-0.25 0.0 0.0" rpy="0 0 0"/>
+             </xacro:if>
+            <geometry>
+              <sphere radius="${screw_collision_radius}"/>
+            </geometry>
+         </collision>
       </link>
-      <gazebo reference="${name}_screw_link">
-        <mu1 value="100"/>
-        <mu2 value="2"/>
-        <kp value="10.0" />
-        <kd value="1.0" />
+      <gazebo reference="${name}_screw_collision_link">
+        <mu1 value="1.1"/>
+        <mu2 value="1.1"/>
+        <kp value="10000.0" />
+        <kd value="100000.0" />
         <material>Gazebo/Grey</material>
       </gazebo>

File: RM3_gazebo/urdf/whisker_snippets.xacro (robot description, xacro)
@@ -12,6 +12,6 @@
   <xacro:property name="base_link_mass" value="0.1"/>
   <xacro:property name="whisker_array_mass" value="2.75"/>
-  <xacro:property name="whisker_revolute_effort_limit" value="10"/>
-  <xacro:property name="whisker_revolute_vel_limit" value="${pi/2}"/>
+  <xacro:property name="whisker_revolute_effort_limit" value="0.01"/>
+  <xacro:property name="whisker_revolute_vel_limit" value="0.0"/>
   <xacro:property name="whisker_x" value="-0.0345"/>
   <xacro:property name="whisker_x_bias" value="0.075"/>
@@ -23,53 +23,69 @@
   <xacro:property name="whisker_collision_box_y" value="0.08"/>
   <xacro:property name="whisker_collision_box_z" value="0.07"/>
+  <xacro:property name="magnet_size_x" value="0.005"/>
+  <xacro:property name="magnet_size_y" value="0.005"/>
+  <xacro:property name="magnet_size_z" value="0.005"/>
+  <xacro:property name="magnet_mass" value="1e-4"/>
  <!-- WHISKER DEFITION -->
   <xacro:macro name="whisker" params="name id parent *origin">
       <!-- Magnet around x axis is connected to whisker array-->
-        <joint name="${name}_magnet_x_${id}" type="revolute">
-        <xacro:insert_block name="origin"/>
-        <parent link="${parent}"/>
-        <child link="${name}_magnet_x_link_${id}"/>
-        <axis xyz="1 0 0" />
-        <limit
+      <joint name="${name}_whisker_fixation_${id}" type="fixed">
+          <xacro:insert_block name="origin"/>
+          <parent link="${parent}"/>
+          <child link="${name}_dummy_${id}"/>
+      </joint>
+      <link name="${name}_dummy_${id}">
+          <inertial>
+          <mass value="${magnet_mass}"/>
+          <inertia
+            ixx="${(1.0/12.0) * magnet_mass * (magnet_size_y ** 2 + magnet_size_z ** 2)}"
+            ixy="0.0"
+            ixz="0.0"
+            iyy="${(1.0/12.0) * magnet_mass * (magnet_size_x ** 2 + magnet_size_z ** 2)}"
+            iyz="0.0"
+            izz="${(1.0/12.0) * magnet_mass * (magnet_size_y ** 2 + magnet_size_x ** 2)}"/>
+          </inertial>
+      </link>
+      <joint name="${name}_magnet_x_${id}" type="revolute">
+          <parent link="${name}_dummy_${id}"/>
+          <child link="${name}_magnet_x_link_${id}"/>
+          <axis xyz="1 0 0" />
+          <limit
           lower="${-pi/2}"
           upper="${pi/2}"
           effort="${whisker_revolute_effort_limit}"
           velocity="${whisker_revolute_vel_limit}" />
-        <dynamics
-          damping="${whisker_damping}"
-          friction="${whisker_friction}" />
-        </joint>
-        <link name="${name}_magnet_x_link_${id}">
-        <inertial>
-        <mass value="0.0005" />
-        <inertia ixx="1.0e-8" ixy="0" ixz="0" iyy="1.0e-8" iyz="0" izz="1.0e-8" />
+          <dynamics
+            damping="${whisker_damping}"
+            friction="${whisker_friction}"
+          />
+      </joint>
+      <link name="${name}_magnet_x_link_${id}">
+          <inertial>
+          <mass value="${magnet_mass}"/>
+          <inertia
+            ixx="${(1.0/12.0) * magnet_mass * (magnet_size_y ** 2 + magnet_size_z ** 2)}"
+            ixy="0.0"
+            ixz="0.0"
+            iyy="${(1.0/12.0) * magnet_mass * (magnet_size_x ** 2 + magnet_size_z ** 2)}"
+            iyz="0.0"
+            izz="${(1.0/12.0) * magnet_mass * (magnet_size_y ** 2 + magnet_size_x ** 2)}"/>
         </inertial>
-        </link>
-        <!-- Magnet around y axis is connected to whisker array-->
-        <joint name="${name}_magnet_y_${id}" type="revolute">
-        <parent link="${name}_magnet_x_link_${id}"/>
-        <child link="${name}_magnet_y_link_${id}"/>
-        <axis xyz="0 1 0" />
-        <limit
-          lower="${-pi/2}"
-          upper="${pi/2}"
-          effort="${whisker_revolute_effort_limit}"
-          velocity="${whisker_revolute_vel_limit}" />
-        <dynamics
-            damping="${whisker_damping}"
-            friction="${whisker_friction}" />
-        </joint>
-        <link name="${name}_magnet_y_link_${id}">
-            <inertial>
-            <mass value="0.0005" />
-            <inertia ixx="1.0e-8" ixy="0" ixz="0" iyy="1.0e-8" iyz="0" izz="1.0e-8" />
-            </inertial>
-        </link>
-      <!-- Whisker fixed on magnet y-->
-      <joint name="${name}_whisker_${id}" type="fixed">
+      </link>
+      <!-- Whisker fixed on magnet x-->
+      <joint name="${name}_whisker_${id}" type="revolute">
           <origin xyz="0 0 0" rpy="0 0 0" />
-          <!-- <parent link="${name}_magnet_y_link_${id}"/> -->
-           <parent link="${name}_magnet_y_link_${id}"/>
+          <parent link="${name}_dummy_${id}"/>
           <child link="${name}_whisker_link_${id}"/>
+          <axis xyz="0 1 0" />
+          <limit
+            lower="${-pi/2} + 0.2"
+            upper="${pi/2} - 0.2"
+            effort="${whisker_revolute_effort_limit}"
+            velocity="${whisker_revolute_vel_limit}" />
+          <dynamics
+              damping="${whisker_damping}"
+              friction="${whisker_friction}"
+              />
       </joint>
       <link name="${name}_whisker_link_${id}">
@@ -79,12 +95,8 @@
             <mass
               value="${whisker_body_mass}" />
-            <!-- <inertia
-              ixx="${1/12 * whisker_body_mass * (3* whisker_radius ** 2 + whisker_length **2 )}" ixy="0" ixz="0"
-              iyy="${1/12 * whisker_body_mass * (3* whisker_radius ** 2 + whisker_length **2 )}" iyz="0"
-              izz="${1/2 * whisker_body_mass * whisker_radius ** 2}" /> -->
               <inertia
-                ixx="${(1/12)*whisker_body_mass*(3*whisker_radius*whisker_radius + whisker_length*whisker_length)}" ixy="0" ixz="0"
-                iyy="${(1/12)*whisker_body_mass*(3*whisker_radius*whisker_radius + whisker_length*whisker_length)}" iyz="0"
-                izz="${(1/2)*whisker_body_mass*whisker_radius*whisker_radius}" />
+                ixx="${(1/12)*whisker_body_mass*(3*whisker_radius**2 + whisker_length**2)}" ixy="0" ixz="0"
+                iyy="${(1/12)*whisker_body_mass*(3*whisker_radius**2 + whisker_length**2)}" iyz="0"
+                izz="${(1/2)*whisker_body_mass*whisker_radius**2}" />
           </inertial>
           <visual>
@@ -92,5 +104,5 @@
                       rpy="0 0 0" />
               <geometry>
-                <cylinder radius="${whisker_radius}" length="${whisker_length-0.01}"/>
+                <cylinder radius="${whisker_radius}" length="${whisker_length}"/>
               </geometry>
           </visual>
@@ -99,18 +111,18 @@
                       rpy="0 0 0" />
               <geometry>
-                <cylinder radius="${whisker_radius}" length="${whisker_length-0.01}"/>
+                <cylinder radius="${whisker_radius}" length="${whisker_length}"/>
               </geometry>
           </collision>
       </link>
-      <!-- <gazebo reference="${name}_magnet_x_${id}">
-      <implicitSpringDamper>true</implicitSpringDamper>
-      <springStiffness>10000</springStiffness>
-      <springReference>0.0</springReference>
+      <gazebo reference="${name}_magnet_x_${id}">
+          <implicitSpringDamper>true</implicitSpringDamper>
+          <springStiffness>5.7</springStiffness>
+          <springReference>0.0</springReference>
       </gazebo>
-      <gazebo reference="${name}_magnet_y_${id}">
-      <implicitSpringDamper>true</implicitSpringDamper>
-      <springStiffness>10000</springStiffness>
-      <springReference>0.0</springReference>
-      </gazebo> -->
+      <gazebo reference="${name}_whisker_${id}">
+          <implicitSpringDamper>true</implicitSpringDamper>
+          <springStiffness>5.7</springStiffness>
+          <springReference>0.0</springReference>
+      </gazebo>
   </xacro:macro>
  <!-- WHISKER ARRAY DEFITION -->
@@ -138,15 +150,6 @@
               </geometry>
           </visual>
-          <collision>
-            <geometry>
-              <box size="${whisker_collision_box_x} ${whisker_collision_box_y} ${whisker_collision_box_z}" />
-            </geometry>
-          </collision>
       </link>
       <gazebo reference="${name}_whisker_array_link">
-        <mu1 value="1"/>
-        <mu2 value="1"/>
-        <kp value="100000.0" />
-        <kd value="1.0" />
         <material>Gazebo/DarkGrey</material>
       </gazebo>

Commit message: Added RGBD camera to the robot. Added xacro:property to enable/disable the camera. Added SLAM mapping launch file with RTABMAP.

File: RM3_gazebo/urdf/RM3_robot.xacro.urdf (robot description, URDF)
Before this commit: robot RM3_robot, 2 links, 1 joints
Joints:
- joint dummy_joint: origin (none) -> xyz=0.0 0.0 -0.32 rpy=0.0 0.0 0.0

File: RM3_gazebo/urdf/screw_snippets.xacro (robot description, xacro)
@@ -31,13 +31,13 @@
         <inertial>
             <xacro:if value="${name == 'BR' or name == 'FL'}">
-                 <origin xyz="-0.17 0.0 0.0" rpy="0 1.57 0"/>
+                 <origin xyz="-0.05 0.0 0.0" rpy="0 1.57 0"/>
             </xacro:if>
             <xacro:if value="${name == 'FR' or name == 'BL'}">
-                 <origin xyz="0.17 0.0 0.0" rpy="0 1.57 0"/>
+                 <origin xyz="0.05 0.0 0.0" rpy="0 1.57 0"/>
             </xacro:if>
           <mass value="${screw_mass / 100}" />
-          <inertia ixx="${(1.0 / 12.0) * screw_mass / 100 * (3 * screw_collision_radius ** 2 + screw_collision_height **2)}"
-                   iyy="${(1.0 / 12.0) * screw_mass / 100 * (3 * screw_collision_radius ** 2 + screw_collision_height **2)}"
-                   izz="${(1.0 / 12.0) * screw_mass / 100 * screw_collision_radius ** 2}"
+          <inertia ixx="${(1.0 / 12.0) * screw_mass / 100 * (3 * 0.01 ** 2 + 0.25 **2)}"
+                   iyy="${(1.0 / 12.0) * screw_mass / 100 * (3 * 0.01 ** 2 + 0.25 **2)}"
+                   izz="${(1.0 / 12.0) * screw_mass / 100 * 0.01 ** 2}"
                    iyz="0.0" ixy="0.0" ixz="0.0"
                     />

File: RM3_gazebo/urdf/sensors.xacro (robot description, xacro)
@@ -5,7 +5,7 @@
 <robot xmlns:xacro="http://www.ros.org/wiki/xacro">
  <!-- IMU DEFITION -->
-  <xacro:macro name="robot_sensors" params="parent">
+  <xacro:macro name="robot_sensors" params="parent enableCamera">
       <gazebo reference="${parent}">
-    <sensor name="br_imu" type="imu">
+      <sensor name="br_imu" type="imu">
         <always_on>true</always_on>
         <update_rate>100</update_rate>
@@ -61,4 +61,42 @@
     </sensor>
     </gazebo>
+    <xacro:if value="${enableCamera == 'enable'}">
+        <gazebo reference="realsense_camera">
+            <sensor name="camera" type="depth">
+                <visualize>true</visualize>
+                <update_rate>60.0</update_rate>
+                <camera name="RS_D455">
+                    <horizontal_fov>1.047198</horizontal_fov>
+                    <image>
+                        <width>640</width>
+                        <height>480</height>
+                        <format>R8G8B8</format>
+                    </image>
+                    <clip>
+                        <near>0.05</near>
+                        <far>3</far>
+                    </clip>
+                </camera>
+                <plugin name="depth_camera_controller" filename="libgazebo_ros_camera.so">
+                    <baseline>0.2</baseline>
+                    <alwaysOn>true</alwaysOn>
+                    <updateRate>0.0</updateRate>
+                    <frame_name>realsense_camera</frame_name>
+                    <pointCloudCutoff>0.5</pointCloudCutoff>
+                    <pointCloudCutoffMax>3.0</pointCloudCutoffMax>
+                    <distortionK1>0</distortionK1>
+                    <distortionK2>0</distortionK2>
+                    <distortionK3>0</distortionK3>
+                    <distortionT1>0</distortionT1>
+                    <distortionT2>0</distortionT2>
+                    <CxPrime>0</CxPrime>
+                    <Cx>0</Cx>
+                    <Cy>0</Cy>
+                    <focalLength>0</focalLength>
+                    <hackBaseline>0</hackBaseline>
+                </plugin>
+            </sensor>
+        </gazebo>
+    </xacro:if>
   </xacro:macro>
 </robot>
