Commit message: Added publishser for Whisker states Adjusted screw locations by 1 cm Adjusted whiskers array naming to make it easier to sort by alphabetical order

File: RM3_gazebo/urdf/whisker_snippets.xacro (robot description, xacro)
@@ -24,8 +24,14 @@
   <xacro:property name="magnet_size_z" value="0.005"/>
   <xacro:property name="magnet_mass" value="1e-4"/>
+<!-- Macro to publish the whisker states -->
+  <xacro:macro name="whisker_feedback" params="joint_name">
+      <joint name="${joint_name}">
+        <state_interface name="position"/>
+      </joint>
+  </xacro:macro>
  <!-- WHISKER DEFITION -->
   <xacro:macro name="whisker" params="name id parent *origin">
       <!-- Magnet around x axis is connected to base_array and rotating around x-->
-      <joint name="${name}_whisker_x_${id}" type="revolute">
+      <joint name="${name}_whisker_${id}_x" type="revolute">
           <xacro:insert_block name="origin"/>
           <parent link="${parent}"/>
@@ -60,5 +66,5 @@
       </link>
       <!-- Whisker fixed on magnet x and rotating around y-->
-      <joint name="${name}_whisker_y_${id}" type="revolute">
+      <joint name="${name}_whisker_${id}_y" type="revolute">
           <origin xyz="0 0 0" rpy="0 0 0" />
           <parent link="${name}_whisker_x_link_${id}"/>
@@ -75,4 +81,11 @@
               />
       </joint>
+      <ros2_control name="GazeboSystem" type="system">
+        <hardware>
+          <plugin>gazebo_ros2_control/GazeboSystem</plugin>
+        </hardware>
+         <xacro:whisker_feedback joint_name="${name}_whisker_${id}_x"/>
+         <xacro:whisker_feedback joint_name="${name}_whisker_${id}_y"/>
+      </ros2_control>
       <link name="${name}_whisker_y_link_${id}">
           <inertial>
@@ -102,10 +115,10 @@
           </collision>
       </link>
-      <gazebo reference="${name}_whisker_x_${id}">
+      <gazebo reference="$${name}_whisker_${id}_x">
           <implicitSpringDamper>true</implicitSpringDamper>
           <springStiffness>1.0</springStiffness>
           <springReference>0.0</springReference>
       </gazebo>
-      <gazebo reference="${name}_whisker_y_${id}">
+      <gazebo reference="${name}_whisker_${id}_y">
           <implicitSpringDamper>true</implicitSpringDamper>
           <springStiffness>1.0</springStiffness>

Commit message: Adjusted whiskers joints damping to reduce their movements noisy behaviour Added an RVIZ config file for the robot in config/Rviz

File: RM3_gazebo/urdf/whisker_snippets.xacro (robot description, xacro)
@@ -9,6 +9,6 @@
   <xacro:property name="whisker_radius" value="0.002"/>
   <xacro:property name="whisker_array_mass" value="2.75"/>
-  <xacro:property name="whisker_damping" value="0.1"/>
-  <xacro:property name="whisker_friction" value="0.01"/>
+  <xacro:property name="whisker_damping" value="2.0"/>
+  <xacro:property name="whisker_friction" value="0.0"/>
   <xacro:property name="whisker_revolute_effort_limit" value="0.1"/>
   <xacro:property name="whisker_revolute_vel_limit" value="${pi/2.0}"/>
@@ -109,16 +109,16 @@
       <gazebo reference="${name}_whisker_${id}_x">
           <implicitSpringDamper>true</implicitSpringDamper>
-          <springStiffness>1.0</springStiffness>
+          <springStiffness>5.7</springStiffness>
           <springReference>0.0</springReference>
       </gazebo>
       <gazebo reference="${name}_whisker_${id}_y">
           <implicitSpringDamper>true</implicitSpringDamper>
-          <springStiffness>1.0</springStiffness>
+          <springStiffness>5.7</springStiffness>
           <springReference>0.0</springReference>
       </gazebo>
       <gazebo reference="${name}_whisker_y_link_${id}">
         <material>Gazebo/White</material>
-        <mu1>0.2</mu1>
-        <mu2>0.2</mu2>
+        <mu1>0</mu1>
+        <mu2>0</mu2>
       </gazebo>
       <ros2_control name="GazeboSystem" type="system">

Commit message: Added Han-sur-Lesse cave in Gazebo: Added possibility to adjust side whiskers and bottom whiskers size in urdf. Reduced physics solver time-step for real-time simulations

File: RM3_gazebo/urdf/whisker_snippets.xacro (robot description, xacro)
@@ -6,5 +6,4 @@
   <xacro:property name="whisker_mesh_file" value="file://$(find rm3_gazebo)/urdf/meshes/whisker.dae"/>
   <xacro:property name="whisker_array_mesh_file" value="file://$(find rm3_gazebo)/urdf/meshes/whisker_array.dae"/>
-  <xacro:property name="whisker_length" value="0.150"/>
   <xacro:property name="whisker_radius" value="0.002"/>
   <xacro:property name="whisker_array_mass" value="2.75"/>
@@ -30,5 +29,5 @@
   </xacro:macro>
  <!-- WHISKER DEFITION -->
-  <xacro:macro name="whisker" params="name id parent *origin">
+  <xacro:macro name="whisker" params="name id parent length *origin">
       <!-- Magnet around x axis is connected to base_array and rotating around x-->
       <joint name="${name}_whisker_${id}_x" type="revolute">
@@ -93,15 +92,15 @@
           </inertial>
           <visual>
-              <origin xyz="0 0 ${whisker_length/2}"
+              <origin xyz="0 0 ${length/2}"
                       rpy="0 0 0" />
               <geometry>
-                <cylinder radius="${whisker_radius}" length="${whisker_length}"/>
+                <cylinder radius="${whisker_radius}" length="${length}"/>
               </geometry>
           </visual>
           <collision>
-              <origin xyz="0 0 ${whisker_length/2}"
+              <origin xyz="0 0 ${length/2}"
                       rpy="0 0 0" />
               <geometry>
-                <cylinder radius="${whisker_radius}" length="${whisker_length}"/>
+                <cylinder radius="${whisker_radius}" length="${length}"/>
               </geometry>
           </collision>
@@ -131,5 +130,5 @@
   </xacro:macro>
  <!-- WHISKER ARRAY DEFITION -->
-  <xacro:macro name="whisker_array" params="name *origin">
+  <xacro:macro name="whisker_array" params="name whisker_length *origin">
       <joint name="${name}_whisker_array" type="fixed">
           <xacro:insert_block name="origin"/>
@@ -159,40 +158,40 @@
       </gazebo>
       <!-- whisker #1 -->
-      <xacro:whisker name="${name}" id = "1" parent= "${name}_whisker_array_link" >
+      <xacro:whisker name="${name}" id = "1" parent= "${name}_whisker_array_link" length = "${whisker_length}">
         <origin xyz="${whisker_x + -3*whisker_x_bias} ${whisker_y} ${whisker_z}"
                 rpy="0 0 0" />
       </xacro:whisker>
       <!-- whisker #2 -->
-      <xacro:whisker name="${name}" id = "2" parent= "${name}_whisker_array_link" >
+      <xacro:whisker name="${name}" id = "2" parent= "${name}_whisker_array_link" length = "${whisker_length}" >
         <origin xyz="${whisker_x + -2*whisker_x_bias} ${whisker_y} ${whisker_z}"
                 rpy="0 0 0" />
       </xacro:whisker>
       <!-- whisker #3 -->
-      <xacro:whisker name="${name}" id = "3" parent= "${name}_whisker_array_link" >
+      <xacro:whisker name="${name}" id = "3" parent= "${name}_whisker_array_link" length = "${whisker_length}">
         <origin xyz="${whisker_x + -whisker_x_bias} ${whisker_y} ${whisker_z}"
                 rpy="0 0 0" />
       </xacro:whisker>
       <!-- whisker #4 -->
-      <xacro:whisker name="${name}" id = "4" parent= "${name}_whisker_array_link" >
+      <xacro:whisker name="${name}" id = "4" parent= "${name}_whisker_array_link" length = "${whisker_length}">
         <origin xyz="${whisker_x + -0*whisker_x_bias} ${whisker_y} ${whisker_z}"
                 rpy="0 0 0" />
       </xacro:whisker>
       <!-- whisker #5 -->
-      <xacro:whisker name="${name}" id = "5" parent= "${name}_whisker_array_link" >
+      <xacro:whisker name="${name}" id = "5" parent= "${name}_whisker_array_link" length = "${whisker_length}">
         <origin xyz="${whisker_x + whisker_x_bias} ${whisker_y} ${whisker_z}"
                 rpy="0 0 0" />
       </xacro:whisker>
       <!-- whisker #6 -->
-      <xacro:whisker name="${name}" id = "6" parent= "${name}_whisker_array_link" >
+      <xacro:whisker name="${name}" id = "6" parent= "${name}_whisker_array_link" length = "${whisker_length}">
         <origin xyz="${whisker_x + 2*whisker_x_bias} ${whisker_y} ${whisker_z}"
                 rpy="0 0 0" />
       </xacro:whisker>
       <!-- whisker #7 -->
-      <xacro:whisker name="${name}" id = "7" parent= "${name}_whisker_array_link" >
+      <xacro:whisker name="${name}" id = "7" parent= "${name}_whisker_array_link" length = "${whisker_length}">
         <origin xyz="${whisker_x + 3*whisker_x_bias} ${whisker_y} ${whisker_z}"
                 rpy="0 0 0" />
       </xacro:whisker>
       <!-- whisker #8 -->
-      <xacro:whisker name="${name}" id = "8" parent= "${name}_whisker_array_link" >
+      <xacro:whisker name="${name}" id = "8" parent= "${name}_whisker_array_link" length = "${whisker_length}">
         <origin xyz="${whisker_x + 4*whisker_x_bias} ${whisker_y} ${whisker_z}"
                 rpy="0 0 0" />

Commit message: Updated whisker arrays meshes Updated number of whisker arrays in the bottom Updated the visualization of point cloud based on new whiskers model Corrected typo in README

File: RM3_gazebo/urdf/whisker_snippets.xacro (robot description, xacro)
@@ -5,5 +5,5 @@
 <robot xmlns:xacro="http://www.ros.org/wiki/xacro">
   <xacro:property name="whisker_mesh_file" value="file://$(find rm3_gazebo)/urdf/meshes/whisker.dae"/>
-  <xacro:property name="whisker_array_mesh_file" value="file://$(find rm3_gazebo)/urdf/meshes/whisker_array.dae"/>
+  <xacro:property name="whisker_array_mesh_file" value="file://$(find rm3_gazebo)/urdf/meshes/whisker_array_thin.dae"/>
   <xacro:property name="whisker_radius" value="0.002"/>
   <xacro:property name="whisker_array_mass" value="2.75"/>
@@ -149,4 +149,5 @@
         </inertial>
           <visual>
+              <origin xyz="0.0 0.0 0.0" rpy="-1.57 0.0 0"/>
               <geometry>
                 <mesh filename="${whisker_array_mesh_file}" scale="1 1 1"/>
